File: headstage_isolation_board_01.sch (EAGLE design)
At the start: 49 parts

Commit message: partially added test points/ dc jack
can now choose between aq board power and external power jack, and
added a few test points
Parts:
- added BOARD_JACK: (no value), jumper:JP2E
- added J1: DC_POWER_JACK-PJ-102AH, RHD2000_eval_board:DC_POWER_JACK-PJ-102AH
- added TP1, TP2, TP3, TP4: TP5P5-25-13, testpad:TP5P5-25-13
Connections:
- new net N$9: TP3A.TP
- new net PWR_JACK: BOARD_JACK.3, J1.PWR, TP4C.TP
- new net VDD_FROM_BOARD: BOARD_JACK.1, S1.VDD, TP4B.TP
- net 5VBOOST: now also TP4A.TP
- net 5V_ISOLATED: now also TP3D.TP
- net GND: now also J1.GND1, J1.GND2, TP4E.TP
- net GND_ISOLATED: now also TP3E.TP
- net VDD33_ISOLATED: now also TP3C.TP
- net VDD_IN: now also BOARD_JACK.2, TP4D.TP; no longer S1.VDD
- net VDD_ISOLATED: now also TP3B.TP
Changed lines of the file:
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@@
 <part name="C18" library="RHD2000_eval_board" deviceset="C" device="_0603" value="100n"/>
 <part name="S3" library="RHD2000_eval_board" deviceset="RHD2000-CABLE-DAQ-SIDE" device=""/>
+<part name="TP1" library="testpad" deviceset="TP5" device="P5-25-13"/>
+<part name="TP2" library="testpad" deviceset="TP5" device="P5-25-13"/>
+<part name="TP3" library="testpad" deviceset="TP5" device="P5-25-13"/>
+<part name="TP4" library="testpad" deviceset="TP5" device="P5-25-13"/>
+<part name="BOARD_JACK" library="jumper" deviceset="JP2E" device=""/>
+<part name="J1" library="RHD2000_eval_board" deviceset="DC_POWER_JACK" device="-PJ-102AH"/>
+<part name="GND12" library="supply1" deviceset="GND" device=""/>
 </parts>
 <sheets>
@@
 <instance part="C18" gate="C" x="99.06" y="-38.1" rot="R90"/>
 <instance part="S3" gate="A" x="-68.58" y="-63.5" rot="R270"/>
+<instance part="TP1" gate="A" x="-22.86" y="-116.84" rot="R180"/>
+<instance part="TP1" gate="B" x="-27.94" y="-116.84" rot="R180"/>
+<instance part="TP1" gate="C" x="-33.02" y="-116.84" rot="R180"/>
+<instance part="TP1" gate="D" x="-38.1" y="-116.84" rot="R180"/>
+<instance part="TP1" gate="E" x="-43.18" y="-116.84" rot="R180"/>
+<instance part="TP2" gate="A" x="160.02" y="-116.84" rot="R180"/>
+<instance part="TP2" gate="B" x="154.94" y="-116.84" rot="R180"/>
+<instance part="TP2" gate="C" x="149.86" y="-116.84" rot="R180"/>
+<instance part="TP2" gate="D" x="144.78" y="-116.84" rot="R180"/>
+<instance part="TP2" gate="E" x="139.7" y="-116.84" rot="R180"/>
+<instance part="TP3" gate="A" x="-55.88" y="88.9"/>
+<instance part="TP3" gate="B" x="-50.8" y="88.9"/>
+<instance part="TP3" gate="C" x="-45.72" y="88.9"/>
+<instance part="TP3" gate="D" x="-40.64" y="88.9"/>
+<instance part="TP3" gate="E" x="-35.56" y="88.9"/>
+<instance part="TP4" gate="A" x="116.84" y="86.36"/>
+<instance part="TP4" gate="B" x="121.92" y="86.36"/>
+<instance part="TP4" gate="C" x="127" y="86.36"/>
+<instance part="TP4" gate="D" x="132.08" y="86.36"/>
+<instance part="TP4" gate="E" x="137.16" y="86.36"/>
+<instance part="BOARD_JACK" gate="1" x="162.56" y="12.7"/>
+<instance part="J1" gate="A" x="205.74" y="-2.54" rot="R180"/>
+<instance part="GND12" gate="1" x="190.5" y="0" rot="R270"/>
 </instances>
 <busses>
@@
 <junction x="40.64" y="-27.94"/>
 </segment>
+<segment>
+<pinref part="TP3" gate="E" pin="TP"/>
+<wire x1="-35.56" y1="86.36" x2="-35.56" y2="83.82" width="0.1524" layer="91"/>
+<label x="-35.56" y="83.82" size="1.778" layer="95"/>
+</segment>
 </net>
 <net name="VDD_ISOLATED" class="0">
@@
 <junction x="-12.7" y="22.86"/>
 </segment>
+<segment>
+<pinref part="TP3" gate="B" pin="TP"/>
+<wire x1="-50.8" y1="86.36" x2="-50.8" y2="83.82" width="0.1524" layer="91"/>
+<label x="-50.8" y="83.82" size="1.778" layer="95" rot="R270"/>
+</segment>
 </net>
 <net name="GND" class="0">
@@
 <junction x="132.08" y="-22.86"/>
 <pinref part="GND11" gate="1" pin="GND"/>
+</segment>
+<segment>
+<pinref part="TP4" gate="E" pin="TP"/>
+<wire x1="137.16" y1="83.82" x2="137.16" y2="81.28" width="0.1524" layer="91"/>
+<label x="137.16" y="81.28" size="1.778" layer="95"/>
+<label x="137.16" y="78.74" size="1.778" layer="95" rot="R270"/>
+</segment>
+<segment>
+<pinref part="J1" gate="A" pin="GND2"/>
+<wire x1="198.12" y1="0" x2="195.58" y2="0" width="0.1524" layer="91"/>
+<pinref part="J1" gate="A" pin="GND1"/>
+<wire x1="198.12" y1="-2.54" x2="195.58" y2="0" width="0.1524" layer="91"/>
+<wire x1="195.58" y1="0" x2="193.04" y2="0" width="0.1524" layer="91"/>
+<pinref part="GND12" gate="1" pin="GND"/>
 </segment>
 </net>
@@
 <junction x="40.64" y="-93.98"/>
 </segment>
+<segment>
+<pinref part="TP3" gate="C" pin="TP"/>
+<wire x1="-45.72" y1="86.36" x2="-45.72" y2="83.82" width="0.1524" layer="91"/>
+<label x="-45.72" y="83.82" size="1.778" layer="95" rot="R270"/>
+</segment>
 </net>
 <net name="N$276" class="0">
@@
 <net name="VDD_IN" class="0">
 <segment>
-<pinref part="S1" gate="A" pin="VDD"/>
-<wire x1="162.56" y1="-38.1" x2="157.48" y2="-38.1" width="0.1524" layer="91"/>
 <pinref part="L2" gate="L" pin="1"/>
 <wire x1="157.48" y1="17.78" x2="147.32" y2="17.78" width="0.1524" layer="91"/>
@@
 <pinref part="C10" gate="C" pin="1"/>
 <wire x1="157.48" y1="30.48" x2="157.48" y2="17.78" width="0.1524" layer="91"/>
-<junction x="157.48" y="17.78"/>
-<wire x1="157.48" y1="17.78" x2="157.48" y2="-38.1" width="0.1524" layer="91"/>
+<wire x1="157.48" y1="17.78" x2="157.48" y2="5.08" width="0.1524" layer="91"/>
+<wire x1="157.48" y1="5.08" x2="162.56" y2="5.08" width="0.1524" layer="91"/>
+<pinref part="BOARD_JACK" gate="1" pin="2"/>
+<wire x1="162.56" y1="5.08" x2="162.56" y2="10.16" width="0.1524" layer="91"/>
+<label x="157.48" y="22.86" size="1.778" layer="95"/>
+<label x="157.48" y="5.08" size="1.778" layer="95" rot="R180"/>
+</segment>
+<segment>
+<pinref part="TP4" gate="D" pin="TP"/>
+<wire x1="132.08" y1="83.82" x2="132.08" y2="81.28" width="0.1524" layer="91"/>
+<label x="132.08" y="81.28" size="1.778" layer="95" rot="R270"/>
 </segment>
 </net>
@@
 <junction x="78.74" y="17.78"/>
 </segment>
+<segment>
+<pinref part="TP4" gate="A" pin="TP"/>
+<wire x1="116.84" y1="83.82" x2="116.84" y2="81.28" width="0.1524" layer="91"/>
+<label x="116.84" y="81.28" size="1.778" layer="95" rot="R270"/>
+</segment>
 </net>
 <net name="N$31" class="0">
@@
 <label x="-76.2" y="22.86" size="1.778" layer="95" rot="R180"/>
 </segment>
+<segment>
+<pinref part="TP3" gate="D" pin="TP"/>
+<wire x1="-40.64" y1="86.36" x2="-40.64" y2="83.82" width="0.1524" layer="91"/>
+<label x="-40.64" y="83.82" size="1.778" layer="95" rot="R270"/>
+</segment>
 </net>
 <net name="N$97" class="0">
@@
 </segment>
 </net>
+<net name="N$9" class="0">
+<segment>
+<pinref part="TP3" gate="A" pin="TP"/>
+<wire x1="-55.88" y1="86.36" x2="-55.88" y2="83.82" width="0.1524" layer="91"/>
+<label x="-55.88" y="83.82" size="1.778" layer="95" rot="R270"/>
+</segment>
+</net>
+<net name="PWR_JACK" class="0">
+<segment>
+<pinref part="J1" gate="A" pin="PWR"/>
+<wire x1="198.12" y1="-5.08" x2="165.1" y2="-5.08" width="0.1524" layer="91"/>
+<pinref part="BOARD_JACK" gate="1" pin="3"/>
+<wire x1="165.1" y1="-5.08" x2="165.1" y2="10.16" width="0.1524" layer="91"/>
+<label x="165.1" y="-2.54" size="1.778" layer="95"/>
+</segment>
+<segment>
+<pinref part="TP4" gate="C" pin="TP"/>
+<wire x1="127" y1="83.82" x2="127" y2="81.28" width="0.1524" layer="91"/>
+<label x="127" y="81.28" size="1.778" layer="95" rot="R270"/>
+</segment>
+</net>
+<net name="VDD_FROM_BOARD" class="0">
+<segment>
+<pinref part="S1" gate="A" pin="VDD"/>
+<wire x1="162.56" y1="-38.1" x2="160.02" y2="-38.1" width="0.1524" layer="91"/>
+<pinref part="BOARD_JACK" gate="1" pin="1"/>
+<wire x1="160.02" y1="-38.1" x2="160.02" y2="10.16" width="0.1524" layer="91"/>
+<label x="160.02" y="0" size="1.778" layer="95" rot="R180"/>
+</segment>
+<segment>
+<pinref part="TP4" gate="B" pin="TP"/>
+<wire x1="121.92" y1="83.82" x2="121.92" y2="81.28" width="0.1524" layer="91"/>
+<label x="121.92" y="81.28" size="1.778" layer="95" rot="R270"/>
+</segment>
+</net>
