File: headstage_isolation_board_01.brd (EAGLE design)
At the start: 50 x 57.4 mm, 57 parts, among them J1 DC_POWER_JACK-PJ-102AH

Commit message: missing brd updates from last commit
Parts:
- moved R5 38.4 mm to (27.7, 34.3), turned to 90 degrees
- moved R6 35.0 mm to (27.2, 29.0)
Routing:
- net MISO2-_ISOLATED: track 26.3 -> 27.9 mm
- net MISO1+_ISOLATED: track 40.3 -> 39.4 mm
- net MISO1-_ISOLATED: track 21.4 -> 22.0 mm
Changed lines of the file:
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@@
 <grid distance="10" unitdist="mil" unit="mil" style="lines" multiple="10" display="yes" altdistance="0.025" altunitdist="inch" altunit="inch"/>
 <layers>
-<layer number="1" name="Top" color="4" fill="1" visible="yes" active="yes"/>
+<layer number="1" name="Top" color="4" fill="1" visible="no" active="yes"/>
 <layer number="2" name="Route2" color="1" fill="3" visible="yes" active="yes"/>
 <layer number="3" name="Route3" color="4" fill="3" visible="yes" active="yes"/>
@@
 <attribute name="VALUE" x="53.34" y="11.049" size="1.27" layer="27" ratio="10"/>
 </element>
-<element name="R5" library="RHD2000_eval_board" package="0603" value="100" x="21.336" y="-3.556"/>
-<element name="R6" library="RHD2000_eval_board" package="0603" value="100" x="21.336" y="-5.588"/>
+<element name="R5" library="RHD2000_eval_board" package="0603" value="100" x="27.686" y="34.29" rot="R90"/>
+<element name="R6" library="RHD2000_eval_board" package="0603" value="100" x="27.178" y="28.956"/>
 </elements>
 <signals>
@@
 <wire x1="28.956" y1="17.018" x2="28.956" y2="25.654" width="0.2032" layer="16"/>
 <wire x1="28.956" y1="25.654" x2="28.448" y2="26.162" width="0.2032" layer="16"/>
-<wire x1="28.448" y1="26.162" x2="28.448" y2="30.988" width="0.2032" layer="16"/>
-<wire x1="28.448" y1="30.988" x2="29.21" y2="31.75" width="0.2032" layer="16"/>
-<wire x1="29.21" y1="31.75" x2="29.21" y2="35.306" width="0.2032" layer="16"/>
+<wire x1="28.448" y1="26.162" x2="28.448" y2="29.21" width="0.2032" layer="16"/>
+<wire x1="28.448" y1="29.21" x2="29.21" y2="29.972" width="0.2032" layer="16"/>
+<wire x1="29.21" y1="29.972" x2="29.21" y2="35.306" width="0.2032" layer="16"/>
 <via x="29.21" y="35.306" extent="1-16" drill="0.6"/>
 <wire x1="29.21" y1="35.306" x2="29.21" y2="35.814" width="0.2032" layer="1"/>
@@
 <wire x1="29.972" y1="36.576" x2="30.988" y2="36.576" width="0.2032" layer="1"/>
 <contactref element="R5" pad="2"/>
-<wire x1="22.1996" y1="-3.556" x2="24.765" y2="16.5735" width="0" layer="19" extent="1-1"/>
+<wire x1="27.686" y1="35.1536" x2="29.21" y2="35.1536" width="0.2032" layer="1"/>
+<wire x1="29.21" y1="35.1536" x2="29.21" y2="35.306" width="0.2032" layer="1"/>
 </signal>
 <signal name="MISO1+_ISOLATED">
@@
 <wire x1="22.1615" y1="17.2085" x2="21.336" y2="17.272" width="0.2032" layer="1"/>
 <wire x1="21.336" y1="17.272" x2="21.336" y2="21.844" width="0.2032" layer="1"/>
-<wire x1="21.336" y1="21.844" x2="26.67" y2="27.178" width="0.2032" layer="1"/>
-<wire x1="26.67" y1="27.178" x2="26.67" y2="32.258" width="0.2032" layer="1"/>
-<wire x1="26.67" y1="32.258" x2="28.194" y2="33.782" width="0.2032" layer="1"/>
-<wire x1="28.194" y1="33.782" x2="29.972" y2="33.782" width="0.2032" layer="1"/>
-<wire x1="29.972" y1="33.782" x2="30.226" y2="34.036" width="0.2032" layer="1"/>
+<wire x1="21.336" y1="21.844" x2="26.162" y2="26.67" width="0.2032" layer="1"/>
+<wire x1="26.162" y1="26.67" x2="26.162" y2="28.956" width="0.2032" layer="1"/>
+<wire x1="26.162" y1="28.956" x2="26.162" y2="29.972" width="0.2032" layer="1"/>
+<wire x1="26.162" y1="29.972" x2="30.226" y2="34.036" width="0.2032" layer="1"/>
 <wire x1="30.226" y1="34.036" x2="30.988" y2="34.036" width="0.2032" layer="1"/>
 <contactref element="TP1" pad="TP-4"/>
@@
 <via x="21.336" y="17.272" extent="1-16" drill="0.5"/>
 <contactref element="R6" pad="1"/>
-<wire x1="20.4724" y1="-5.588" x2="23.876" y2="11.176" width="0" layer="19" extent="1-1"/>
+<wire x1="26.3144" y1="28.956" x2="26.162" y2="28.956" width="0.2032" layer="1"/>
 </signal>
 <signal name="MISO1-_ISOLATED">
@@
 <wire x1="27.8765" y1="17.2085" x2="27.94" y2="17.272" width="0.2032" layer="1"/>
 <via x="27.94" y="17.272" extent="1-16" drill="0.6"/>
-<wire x1="27.94" y1="17.272" x2="27.94" y2="32.258" width="0.2032" layer="16"/>
-<wire x1="27.94" y1="32.258" x2="28.448" y2="32.766" width="0.2032" layer="16"/>
-<via x="28.448" y="32.766" extent="1-16" drill="0.6"/>
-<wire x1="28.448" y1="32.766" x2="30.988" y2="32.766" width="0.2032" layer="1"/>
+<wire x1="27.94" y1="17.272" x2="27.94" y2="29.972" width="0.2032" layer="16"/>
+<wire x1="27.94" y1="29.972" x2="28.448" y2="30.48" width="0.2032" layer="16"/>
+<via x="28.448" y="30.48" extent="1-16" drill="0.6"/>
+<wire x1="28.448" y1="30.48" x2="30.734" y2="32.766" width="0.2032" layer="1"/>
+<wire x1="30.734" y1="32.766" x2="30.988" y2="32.766" width="0.2032" layer="1"/>
 <contactref element="R6" pad="2"/>
-<wire x1="22.1996" y1="-5.588" x2="24.765" y2="17.2085" width="0" layer="19" extent="1-1"/>
+<wire x1="28.0416" y1="28.956" x2="28.067" y2="28.956" width="0.2032" layer="1"/>
+<wire x1="28.067" y1="28.956" x2="28.067" y2="30.099" width="0.2032" layer="1"/>
+<wire x1="28.067" y1="30.099" x2="28.448" y2="30.099" width="0.2032" layer="1"/>
+<wire x1="28.448" y1="30.099" x2="28.448" y2="30.48" width="0.2032" layer="1"/>
 </signal>
 <signal name="MISO2+_ISOLATED">
@@
 <contactref element="S3" pad="B5"/>
 <wire x1="30.988" y1="35.306" x2="30.226" y2="35.306" width="0.2032" layer="1"/>
-<wire x1="30.226" y1="35.306" x2="29.21" y2="34.29" width="0.2032" layer="1"/>
-<wire x1="29.21" y1="34.29" x2="27.432" y2="34.29" width="0.2032" layer="1"/>
-<wire x1="27.432" y1="34.29" x2="26.67" y2="33.528" width="0.2032" layer="1"/>
-<via x="26.67" y="33.528" extent="1-16" drill="0.6"/>
-<wire x1="26.67" y1="33.528" x2="26.67" y2="27.178" width="0.2032" layer="16"/>
-<wire x1="26.67" y1="27.178" x2="23.876" y2="24.384" width="0.2032" layer="16"/>
+<wire x1="30.226" y1="35.306" x2="28.448" y2="33.528" width="0.2032" layer="1"/>
+<wire x1="28.448" y1="33.528" x2="27.686" y2="33.528" width="0.2032" layer="1"/>
+<wire x1="27.686" y1="33.528" x2="26.67" y2="33.528" width="0.2032" layer="1"/>
+<wire x1="26.67" y1="33.528" x2="26.162" y2="33.02" width="0.2032" layer="1"/>
+<via x="26.162" y="33.02" extent="1-16" drill="0.6"/>
+<wire x1="26.162" y1="33.02" x2="26.162" y2="26.67" width="0.2032" layer="16"/>
+<wire x1="26.162" y1="26.67" x2="23.876" y2="24.384" width="0.2032" layer="16"/>
 <wire x1="23.876" y1="24.384" x2="23.876" y2="18.288" width="0.2032" layer="16"/>
 <wire x1="23.876" y1="18.288" x2="22.098" y2="16.51" width="0.2032" layer="16"/>
@@
 <wire x1="23.1775" y1="16.51" x2="23.622" y2="16.5735" width="0.2032" layer="1"/>
 <contactref element="R5" pad="1"/>
-<wire x1="20.4724" y1="-3.556" x2="22.098" y2="16.51" width="0" layer="19" extent="1-16"/>
+<wire x1="27.686" y1="33.4264" x2="27.686" y2="33.528" width="0.2032" layer="1"/>
 </signal>
 <signal name="SCLK-">
@@
 <vertex x="40.64" y="65.786"/>
 <vertex x="15.748" y="62.23"/>
-<vertex x="15.748" y="-2.286"/>
+<vertex x="15.494" y="3.048"/>
 <vertex x="40.64" y="-2.286"/>
 </polygon>
@@
 <vertex x="40.64" y="65.786"/>
 <vertex x="16.764" y="63.246"/>
-<vertex x="17.272" y="0.508"/>
+<vertex x="16.256" y="1.016"/>
 <vertex x="40.64" y="-2.286"/>
 </polygon>
@@
 <wire x1="25.019" y1="42.1894" x2="25.019" y2="41.529" width="0.2032" layer="1"/>
 <wire x1="25.019" y1="41.529" x2="26.924" y2="39.624" width="0.2032" layer="1"/>
-<wire x1="26.924" y1="39.624" x2="26.924" y2="35.56" width="0.2032" layer="1"/>
+<wire x1="26.924" y1="39.624" x2="26.924" y2="36.322" width="0.2032" layer="1"/>
 <wire x1="23.434" y1="49.102" x2="23.434" y2="48.702" width="0.2032" layer="1"/>
 <wire x1="23.434" y1="48.702" x2="23.876" y2="48.26" width="0.2032" layer="1"/>
@@
 <wire x1="28.956" y1="49.276" x2="30.353" y2="49.276" width="0.2032" layer="1"/>
 <wire x1="30.353" y1="49.276" x2="30.48" y2="49.403" width="0.2032" layer="1"/>
-<wire x1="26.924" y1="35.56" x2="24.892" y2="33.528" width="0.2032" layer="1"/>
-<wire x1="24.892" y1="33.528" x2="24.892" y2="33.02" width="0.2032" layer="1"/>
+<wire x1="26.924" y1="36.322" x2="24.892" y2="34.29" width="0.2032" layer="1"/>
+<wire x1="24.892" y1="34.29" x2="24.892" y2="33.02" width="0.2032" layer="1"/>
 <wire x1="24.718" y1="32.954" x2="24.318" y2="32.954" width="0.2032" layer="1"/>
 <wire x1="24.318" y1="32.954" x2="23.876" y2="32.512" width="0.2032" layer="1"/>
@@
 <contactref element="5VD" pad="4"/>
 <contactref element="C52" pad="1"/>
-<wire x1="28.8036" y1="41.402" x2="28.702" y2="40.386" width="0.2032" layer="1"/>
+<wire x1="28.8036" y1="41.402" x2="28.956" y2="40.64" width="0.2032" layer="1"/>
 <wire x1="22.018" y1="32.954" x2="22.018" y2="33.862" width="0.2032" layer="1"/>
 <wire x1="22.018" y1="33.862" x2="21.844" y2="34.036" width="0.2032" layer="1"/>
@@
 <wire x1="25.908" y1="39.878" x2="28.194" y2="39.878" width="0.2032" layer="16"/>
 <via x="28.194" y="39.878" extent="1-16" drill="0.6"/>
-<wire x1="28.194" y1="39.878" x2="28.702" y2="40.386" width="0.2032" layer="1"/>
+<wire x1="28.194" y1="39.878" x2="28.956" y2="40.64" width="0.2032" layer="1"/>
 </signal>
 <signal name="N$108">
